File: AvionicsPower.kicad_pcb (KiCad board)
At the start: 2 copper layers, 60 x 56.1 mm, 65 parts, among them J2 Conn_01x02, P1 USB_C_Plug, Q1 AO3400A, Q2 AO3400A, Q3 NCE8205, U3 RP2040, U4 AP2112K-3.3, U5 W25Q128JVS, U6 Shenzhen Fuman Elec FM2113, U7 SN65HVD230DR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

Commit message: basic layout
Parts:
- added C2: 10uf, PCM_JLCPCB:C_0805, F.Cu at (129.3, 35.9)
- added R23: 200Ω, PCM_JLCPCB:R_0402, F.Cu at (135.2, 48.1)
- added R3: 250k, PCM_JLCPCB:R_1206, F.Cu at (129.9, 32.7)
- added R4: 10kΩ, PCM_JLCPCB:R_0805, F.Cu at (184.8, -0.22)
- moved Q1 71.3 mm to (189.5, 7.25)
- moved C13 62.4 mm to (142.2, 57.7)
- moved C15 62.4 mm to (143.9, 59.6)
- moved R10 62.4 mm to (140.2, 71.0)
- moved C10 62.4 mm to (143.9, 64.3)
- moved C11 62.4 mm to (134.6, 64.4)
- moved C12 62.4 mm to (134.6, 60.8)
- moved C14 62.4 mm to (143.1, 57.7)
- moved C16 62.4 mm to (139.5, 57.6)
- moved C17 62.4 mm to (137.5, 52.4)
- moved C18 62.4 mm to (137.8, 72.2)
- moved C19 62.4 mm to (138.1, 67.8)
- moved C6 62.4 mm to (138.6, 57.6)
- moved C7 62.4 mm to (141.3, 57.7)
- moved C8 62.4 mm to (141.5, 69.0)
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Connections:
- J2 pad 1: +1S LiPo -> -1S LiPo
- J2 pad 2: -1S LiPo -> +1S LiPo
Routing:
- net -1S LiPo: track 0.00 -> 9.23 mm
- net /DP: track 0.00 -> 7.42 mm
- net GND: track 36.8 -> 44.2 mm, vias 22 -> 26
- net /DN: track 0.00 -> 7.34 mm
- net Net-(Q3-G2): track 0.00 -> 6.82 mm, vias 0 -> 2
- net +1S LiPo: track 0.00 -> 4.42 mm
- net Net-(Q3-D1/D2-Pad2): track 0.00 -> 2.70 mm
- net +5V: track 0.00 -> 2.56 mm
- net Net-(U6-VDD): track 0.00 -> 2.30 mm
- net Net-(D3-Pad1): track 0.00 -> 1.94 mm
- net Net-(P1-CC2): track 0.00 -> 1.64 mm
- net Net-(P1-CC1): track 0.00 -> 1.63 mm
- net Net-(Q3-G1): track 0.00 -> 1.46 mm
- net Net-(U6-CS): track 0.00 -> 1.40 mm
